Commit message: Fixed link name.

File: code/urdf_tutorial/urdf/robot_0.urdf (robot description, URDF)
Before this commit: robot robot_0, 2 links, 1 joints
Joints:
- removed joint base_to_astra_camera
- added joint base_to_astra_camera_link: type fixed, parent base_link, child astra_camera_link

Commit message: Added pcl detection of objects (has to be run separately).

File: code/urdf_tutorial/urdf/robot_0.urdf (robot description, URDF)
Before this commit: robot robot_0, 2 links, 1 joints
Links:
- removed link astra_camera_link
- added link camera_link; visual box size=0.6 0.1 0.2
Joints:
- joint base_to_astra_camera_link: child astra_camera_link -> camera_link

Commit message: Modified rViz skeleton image. Added screenshot of pointed ray.

File: code/urdf_tutorial/urdf/robot_0.urdf (robot description, URDF)
Before this commit: robot robot_0, 2 links, 1 joints
Links:
- link base_link: geometry visual cylinder length=1 radius=0.1
- link camera_link: geometry visual box size=0.2 0.1 0.2

Commit message: Debugged object detection (floor plane). Modified grip gesture (both hands) to minimize noise errors.

File: code/urdf_tutorial/urdf/robot_0.urdf (robot description, URDF)
Before this commit: robot robot_0, 2 links, 1 joints
Links:
- link base_link: geometry visual cylinder length=0.8 radius=0.1
