Commit message: Updated UR settings.

File: code_robot/src/impakt_pkg/impakt_robot.urdf.xacro (robot description, xacro)
@@ -788,5 +788,5 @@
            link/frame) to introduce the necessary rotation over Z (of pi rad).
       -->
-        <origin rpy="0 0 3.141592653589793" xyz="0 0 0" />
+        <origin rpy="0 0 1.5707963267948966" xyz="0 0 0" />
     </joint>
     <joint name="ur5_shoulder_pan_joint" type="revolute">

File: code_robot/src/ur_description/urdf/inc/ur_common.xacro (robot description, xacro)
@@ -26,15 +26,12 @@
   <!--  TODO: remove params -->
   <xacro:macro name="read_model_data" params="
-  joint_limits_parameters_file:='$(find impakt_pkg)/joint_limits.yaml'
-   kinematics_parameters_file:='$(find impakt_pkg)/default_kinematics.yaml'
-   physical_parameters_file:='$(find impakt_pkg)/physical_parameters.yaml'
-   visual_parameters_file:='$(find impakt_pkg)/visual_parameters.yaml'
+  joint_limits_parameters_file kinematics_parameters_file physical_parameters_file visual_parameters_file
    ">
     <!-- Read .yaml files from disk, load content into properties -->
     <!--xacro:property name="config_joint_limit_parameters" value="${xacro.load_yaml('./joint_limits.yaml')}"/-->
-    <xacro:property name="config_joint_limit_parameters" value="${xacro.load_yaml('./joint_limits.yaml')}"/>
-    <xacro:property name="config_kinematics_parameters"  value="${xacro.load_yaml('./default_kinematics.yaml')}"/>
-    <xacro:property name="config_physical_parameters"    value="${xacro.load_yaml('./physical_parameters.yaml')}"/>
-    <xacro:property name="config_visual_parameters"      value="${xacro.load_yaml('./visual_parameters.yaml')}"/>
+    <xacro:property name="config_joint_limit_parameters" value="${xacro.load_yaml('../config/ur5/joint_limits.yaml')}"/>
+    <xacro:property name="config_kinematics_parameters"  value="${xacro.load_yaml('../config/ur5/default_kinematics.yaml')}"/>
+    <xacro:property name="config_physical_parameters"    value="${xacro.load_yaml('../config/ur5/physical_parameters.yaml')}"/>
+    <xacro:property name="config_visual_parameters"      value="${xacro.load_yaml('../config/ur5/visual_parameters.yaml')}"/>
     <!-- Extract subsections from yaml dictionaries -->
     <xacro:property name="sec_limits" value="${config_joint_limit_parameters['joint_limits']}"/>
