Commit message: Added end effector. Modified reference to joint_limits.

File: code_robot/src/ur_description/urdf/impakt_wsg_50.urdf.xacro (robot description, xacro)
@@ -1,47 +1,1204 @@
-<?xml version="1.0"?>
-<robot  xmlns:sensor="http://playerstage.sourceforge.net/gazebo/xmlschema/#sensor"
-	xmlns:controller="http://playerstage.sourceforge.net/gazebo/xmlschema/#controller"
-	xmlns:interface="http://playerstage.sourceforge.net/gazebo/xmlschema/#interface"
-        xmlns:xacro="http://ros.org/wiki/xacro"
-	name="wsg_50_coupler">
-<xacro:include filename="$(find impakt_pkg)/impakt_robot.urdf.xacro" />
-<xacro:include filename="$(find wsg_50_simulation)/urdf/wsg_50.urdf.xacro" />
-  <!-- Wsg Coupler -->
-  <!--  + Height added by the coupler: 8mm -->
-  <!--  + Reference frame: at the middle (4mm) -->
-  <link name="wsg_coupler">
-    <inertial>
-      <origin xyz="2.073e-05   1.45286e-03  -1.1049e-03" rpy="0 0 0" />
-      <mass value="0.168" />
-      <inertia ixx="6.69695624e-05" ixy="5.21511788e-09" ixz="-2.74383009e-08"
-               iyy="7.85088161e-05" iyz="5.41105193e-07" izz="1.41819717e-04"/>
-    </inertial>
-  </link>
-  <joint name="wsg_coupler_joint" type="fixed">
-    <origin xyz="0 0 0.004" rpy="0 0 0" />
-    <parent link="ur5_tool0"/>
-    <child link="wsg_coupler"/>
-  </joint>
-  <gazebo reference="wsg_coupler">
-    <mu1>0.9</mu1>
-    <mu2>0.9</mu2>
-    <material>Gazebo/FlatBlack</material>
-  </gazebo>
-  <!-- Attach the wsg gripper -->
-  <xacro:wsg_50_xacro parent="wsg_coupler" finger_length="0.023" finger_tip="0" name="wsg_50">
-    <origin xyz="0 0 0.004" rpy="0 0 0"/>
-  </xacro:wsg_50_xacro>
-  <!-- Gazebo FT sensor plugin -->
-  <gazebo reference="wrist_3_joint">
-    <provideFeedback>true</provideFeedback>
-  </gazebo>
-  <gazebo>
-    <plugin name="ft_sensor_plugin" filename="libgazebo_ros_ft_sensor.so">
-      <updateRate>250.0</updateRate>
-      <topicName>ft_sensor/raw</topicName>
-      <gaussianNoise>0.0</gaussianNoise>
-      <jointName>wrist_3_joint</jointName>
-    </plugin>
-  </gazebo>
-  <!-- Gazebo grasping plugin -->
+<?xml version="1.0" ?>
+<!-- =================================================================================== -->
+<!-- |    This document was autogenerated by xacro from /home/lada/Desktop/catkin_2024/ws/src/ur_description/urdf/impakt_wsg_50.urdf.xacro | -->
+<!-- |    EDITING THIS FILE BY HAND IS NOT RECOMMENDED                                 | -->
+<!-- =================================================================================== -->
+<robot name="wsg_50_coupler" xmlns:controller="http://playerstage.sourceforge.net/gazebo/xmlschema/#controller" xmlns:interface="http://playerstage.sourceforge.net/gazebo/xmlschema/#interface" xmlns:sensor="http://playerstage.sourceforge.net/gazebo/xmlschema/#sensor">
+    <!--
+    This is a top-level xacro instantiating the Gazebo-specific version of the
+    'ur_robot' macro (ie: 'ur_robot_gazebo') and passing it values for all its
+    required arguments.
+    This file should be considered the Gazebo-specific variant of the file
+    with the same name in the ur_description package. It accepts the same
+    arguments, but instead of configuring everything for a real robot, will
+    generate a Gazebo-compatible URDF with a ros_control hardware_interface
+    attached to it.
+    Only use this top-level xacro if you plan on spawning the robot in Gazebo
+    'by itself', without any gripper or any other geometry attached.
+    If you need to attach an end-effector, camera or need to integrate the
+    robot into a larger workcell and want to spawn that as a single entity in
+    Gazebo, DO NOT EDIT THIS FILE.
+    Instead: create a new top-level xacro, give it a proper name, include the
+    required '.xacro' files, instantiate the models (ie: call the macros) and
+    connect everything by adding the appropriate joints.
+  -->
+    <!--
+    Import main macro.
+    NOTE: this imports the Gazebo-wrapper main macro, NOT the regular
+          xacro macro (which is hosted by ur_description).
+  -->
+    <gazebo>
+        <plugin filename="libgazebo_ros_diff_drive.so" name="differential_drive_controller">
+            <alwaysOn>true</alwaysOn>
+            <updateRate>40</updateRate>
+            <legacyMode>false</legacyMode>
+            <leftJoint>wheel_left_joint</leftJoint>
+            <rightJoint>wheel_right_joint</rightJoint>
+            <wheelSeparation>0.592</wheelSeparation>
+            <wheelDiameter>0.260</wheelDiameter>
+            <torque>20</torque>
+            <commandTopic>cmd_vel</commandTopic>
+            <odometryTopic>odom</odometryTopic>
+            <odometryFrame>odom</odometryFrame>
+            <robotBaseFrame>base_link</robotBaseFrame>
+            <publishWheelTF>false</publishWheelTF>
+            <publishWheelJointState>true</publishWheelJointState>
+            <rosDebugLevel>na</rosDebugLevel>
+            <wheelAcceleration>0</wheelAcceleration>
+            <wheelTorque>5</wheelTorque>
+            <odometrySource>world</odometrySource>
+            <publishTf>true</publishTf>
+            <publishOdomTF>true</publishOdomTF>
+        </plugin>
+        <plugin name="gazebo_ros_control">
+            <robotNamespace>/</robotNamespace>
+        </plugin>
+    </gazebo>
+    <gazebo reference="lidar_1_link">
+        <sensor name="lidar_1_link" type="ray">
+            <pose>0 0 0 0 0 0</pose>
+            <visualize>false</visualize>
+            <update_rate>100</update_rate>
+            <ray>
+                <scan>
+                    <horizontal>
+                        <samples>720</samples>
+                        <resolution>1</resolution>
+                        <min_angle>-1.48353</min_angle>
+                        <max_angle>1.48353</max_angle>
+                    </horizontal>
+                </scan>
+                <range>
+                    <min>0.10</min>
+                    <max>30.0</max>
+                    <resolution>0.05</resolution>
+                </range>
+                <noise>
+                    <type>gaussian</type>
+                    <!-- Noise parameters based on published spec for Hokuyo laser
+                   achieving "+-30mm" accuracy at range < 10m.  A mean of 0.0m and
+                   stddev of 0.01m will put 99.7% of samples within 0.03m of the true
+                   reading. -->
+                    <mean>0.0</mean>
+                    <stddev>0.01</stddev>
+                </noise>
+            </ray>
+            <plugin filename="libgazebo_ros_laser.so" name="lidar_1_link">
+                <topicName>lidar_1/scan_filtered</topicName>
+                <frameName>lidar_1_link</frameName>
+            </plugin>
+        </sensor>
+    </gazebo>
+    <!-- IMU sensor -->
+    <gazebo reference="imu_link">
+        <gravity>true</gravity>
+        <sensor name="imu_sensor" type="imu">
+            <always_on>true</always_on>
+            <update_rate>100</update_rate>
+            <visualize>true</visualize>
+            <topic>__default_topic__</topic>
+            <plugin filename="libgazebo_ros_imu_sensor.so" name="imu_plugin">
+                <topicName>imu</topicName>
+                <bodyName>imu_link</bodyName>
+                <updateRateHZ>10.0</updateRateHZ>
+                <gaussianNoise>0.0</gaussianNoise>
+                <xyzOffset>0 0 0</xyzOffset>
+                <rpyOffset>0 0 0</rpyOffset>
+                <frameName>imu_link</frameName>
+            </plugin>
+            <pose>0 0 0 0 0 0</pose>
+        </sensor>
+    </gazebo>
+    <!-- Ultrasonic sensors -->
+    <gazebo reference="us_1_link">
+        <!-- Visuals / Collisions omitted for this example -->
+        <sensor name="range" type="ray">
+            <ray>
+                <scan>
+                    <horizontal>
+                        <samples>1</samples>
+                        <resolution>1.0</resolution>
+                        <min_angle>-0.01</min_angle>
+                        <max_angle>0.01</max_angle>
+                    </horizontal>
+                    <vertical>
+                        <samples>1</samples>
+                        <resolution>1</resolution>
+                        <min_angle>-0.01</min_angle>
+                        <max_angle>0.01</max_angle>
+                    </vertical>
+                </scan>
+                <range>
+                    <min>0.01</min>
+                    <max>3.75</max>
+                    <resolution>0.02</resolution>
+                </range>
+            </ray>
+            <plugin filename="libgazebo_ros_range.so" name="libgazebo_ros_range">
+                <gaussianNoise>0.005</gaussianNoise>
+                <alwaysOn>true</alwaysOn>
+                <updateRate>50</updateRate>
+                <topicName>ultrasonic/us1</topicName>
+                <frameName>us_1_link</frameName>
+                <radiation>SONAR</radiation>
+                <fov>0.2967</fov>
+            </plugin>
+        </sensor>
+    </gazebo>
+    <!-- camera -->
+    <gazebo reference="camera_link">
+        <sensor name="camera1" type="camera">
+            <update_rate>30.0</update_rate>
+            <camera name="head">
+                <horizontal_fov>1.3962634</horizontal_fov>
+                <image>
+                    <width>800</width>
+                    <height>800</height>
+                    <format>R8G8B8</format>
+                </image>
+                <clip>
+                    <near>0.02</near>
+                    <far>300</far>
+                </clip>
+                <noise>
+                    <type>gaussian</type>
+                    <!-- Noise is sampled independently per pixel on each frame.
+               That pixel's noise value is added to each of its color
+               channels, which at that point lie in the range [0,1]. -->
+                    <mean>0.0</mean>
+                    <stddev>0.007</stddev>
+                </noise>
+            </camera>
+            <plugin filename="libgazebo_ros_camera.so" name="camera_controller">
+                <alwaysOn>true</alwaysOn>
+                <updateRate>0.0</updateRate>
+                <cameraName>camera1</cameraName>
+                <imageTopicName>image_raw</imageTopicName>
+                <cameraInfoTopicName>camera_info</cameraInfoTopicName>
+                <frameName>camera_link</frameName>
+                <hackBaseline>0.07</hackBaseline>
+                <distortionK1>0.0</distortionK1>
+                <distortionK2>0.0</distortionK2>
+                <distortionK3>0.0</distortionK3>
+                <distortionT1>0.0</distortionT1>
+                <distortionT2>0.0</distortionT2>
+            </plugin>
+        </sensor>
+    </gazebo>
+    <!-- <gazebo>
+  <plugin name="gazebo_ros_control" filename="libgazebo_ros_control.so">
+ <legacyModeNS> false </legacyModeNS>
+  <robotParam>/robot_description</robotParam>
+       <robotSimType>gazebo_ros_control/DefaultRobotHWSim</robotSimType>
+  </plugin>
+</gazebo> -->
+    <!--++++++++++++++++++++++++++++++base_link++++++++++++++++++++++++++++++++++++++++++++++++++++-->
+    <!--++++++++++++++++++++body++++++++++++++++++++++++++++-->
+    <!-- SENSORS -->
+    <!-- Sick S300 - Comment/Uncomment if required  -->
+    <!-- Microscan - Comment/Uncomment if required -->
+    <!-- <xacro:include filename="$(find neo_simulation)/robots/mp_500/xacros/micro_scan.xacro" /> -->
+    <!-- USS, IMU and Camera- Comment/Uncomment if required  -->
+    <!-->
+  <xacro:include filename="$(find neo_simulation)/robots/mp_500/xacros/imu.xacro" />
+  <xacro:include filename="$(find neo_simulation)/robots/mp_500/xacros/ultrasonic.xacro" />
+  <xacro:include filename="$(find neo_simulation)/robots/mp_500/xacros/camera.xacro" />
+  <-->
+    <link name="base_link" />
+    <joint name="above_body_box_joint" type="fixed">
+        <origin rpy="0 0 0" xyz="-0.3 0 0.505" />
+        <axis xyz="0 0 0" />
+        <parent link="base_footprint" />
+        <child link="above_body_box_link" />
+    </joint>
+    <link name="above_body_box_link">
+        <inertial>
+            <mass value="15" />
+            <origin rpy="0 0 0" xyz="0 0 0" />
+            <inertia ixx="0" ixy="0.0" ixz="0.0" iyy="0" iyz="0.0" izz="0" />
+        </inertial>
+        <visual>
+            <origin rpy="0 0 0" xyz="0 0 0" />
+            <geometry>
+                <box size="0.23 0.4 0.3" />
+            </geometry>
+            <material name="grey">
+                <color rgba="0.7 0.7 0.7 1" />
+            </material>
+        </visual>
+        <collision>
+            <origin rpy="0 0 0" xyz="0 0 0" />
+            <geometry>
+                <box size="0.23 0.4 0.3" />
+            </geometry>
+        </collision>
+    </link>
+    <gazebo reference="above_body_box_link">
+        <material>Gazebo/Grey</material>
+    </gazebo>
+    <joint name="above_body_platform_joint" type="fixed">
+        <origin rpy="0 0 0" xyz="-0.05 0 0.4" />
+        <axis xyz="0 0 0" />
+        <parent link="base_footprint" />
+        <child link="above_body_platform_link" />
+    </joint>
+    <link name="above_body_platform_link">
+        <inertial>
+            <mass value="5.1" />
+            <origin rpy="0 0 0" xyz="0 0 0" />
+            <inertia ixx="0" ixy="0.0" ixz="0.0" iyy="0" iyz="0.0" izz="0" />
+        </inertial>
+        <visual>
+            <origin rpy="0 0 0" xyz="0 0 0" />
+            <geometry>
+                <box size="0.26 0.26 0.15" />
+            </geometry>
+            <material name="black">
+                <color rgba="1 1 1 1" />
+            </material>
+        </visual>
+        <collision>
+            <origin rpy="0 0 0" xyz="0 0 0" />
+            <geometry>
+                <box size="0.26 0.26 0.15" />
+            </geometry>
+        </collision>
+    </link>
+    <gazebo reference="above_body_platform_link">
+        <material>Gazebo/Black</material>
+    </gazebo>
+    <joint name="base_footprint_joint" type="fixed">
+        <origin rpy="0 0 0" xyz="0 0 0" />
+        <axis xyz="0 0 -1" />
+        <!-- <limit effort="1000.0" lower="-1e+16" upper="1e+16" velocity="3.5"/> -->
+        <joint_properties damping="1" friction="1" />
+        <parent link="base_link" />
+        <child link="base_footprint" />
+    </joint>
+    <link name="base_footprint">
+        <inertial>
+            <mass value="64.5" />
+            <origin rpy="0 0 0" xyz="0 0 0" />
+            <inertia ixx="1.71402" ixy="0.0" ixz="0.0" iyy="0.8856" iyz="0.0" izz="2.5725" />
+        </inertial>
+        <visual name="body">
+            <origin rpy="0 0 1.570796" xyz="0.0 0.0 0" />
+            <geometry>
+                <mesh filename="package://neo_simulation/robots/mp_500/meshes/MP-500-BODY.dae" scale="0.001 0.001 0.001" />
+            </geometry>
+        </visual>
+        <collision name="body_collision">
+            <origin rpy=" 0 0. 1.570796" xyz="0.0 0.0 0.0" />
+            <geometry>
+                <mesh filename="package://neo_simulation/robots/mp_500/meshes/MP-500-BODY.dae" scale="0.001 0.001 0.001" />
+            </geometry>
+        </collision>
+    </link>
+    <joint name="caster_wheel_joint" type="fixed">
+        <origin rpy="-1.570796 0 1.570796 " xyz="-0.43 0. 0.176" />
+        <axis xyz="0 -1 0" />
+        <limit effort="1000.0" lower="-1e+16" upper="1e+16" velocity="3.5" />
+        <parent link="base_footprint" />
+        <child link="caster_wheel_link" />
+        <joint_properties damping="1.0" friction="1.0" />
+    </joint>
+    <link name="caster_wheel_link" type="wheel">
+        <inertial>
+            <mass value="1.82362" />
+            <inertia ixx="0.00499743171" ixy="0.00000004464" ixz="-0.00000002245" iyy="0.00499741733" iyz="0.00000000164" izz="0.00839239692" />
+            <origin rpy="0 0 0" xyz="0 0 0" />
+        </inertial>
+        <visual name="castor_wheel">
+            <origin rpy="0 0 0" xyz="0 0 0" />
+            <geometry>
+                <mesh filename="package://neo_simulation/robots/mp_500/meshes/MP-500-WHEEL.dae" scale="0.001 0.001 0.001" />
+            </geometry>
+        </visual>
+        <collision>
+            <origin rpy="0 0 0" xyz="0 0 0" />
+            <geometry>
+                <mesh filename="package://neo_simulation/robots/mp_500/meshes/MP-500-WHEEL.dae" scale="0.001 0.001 0.001" />
+            </geometry>
+        </collision>
+    </link>
+    <gazebo reference="caster_wheel_link">
+        <kp>8000.0</kp>
+        <kd>1460.0</kd>
+        <mu1>0.5</mu1>
+        <mu2>0.2</mu2>
+        <fdir1>1 0 0</fdir1>
+        <maxVel>3.0</maxVel>
+        <minDepth>0.00</minDepth>
+    </gazebo>
+    <joint name="wheel_right_joint" type="revolute">
+        <origin rpy="0 0 -1.570796" xyz="0. -0.25 0.13" />
+        <limit effort="1000.0" lower="-1e+16" upper="1e+16" velocity="3.5" />
+        <axis xyz="-1 0 0" />
+        <joint_properties damping="0" friction="0.0" />
+        <parent link="base_link" />
+        <child link="wheel_right_link" />
+    </joint>
+    <link name="wheel_right_link" type="wheel">
+        <inertial>
+            <origin rpy="0 0 0" xyz="0 0 0" />
+            <mass value="1.82362" />
+            <inertia ixx="0.00399743171" ixy="0.00000004464" ixz="-0.00000002245" iyy="0.00399741733" iyz="-0.00000000164" izz="0.00739239692" />
+        </inertial>
+        <visual>
+            <origin rpy="0 0 0" xyz="0 0 0" />
+            <geometry>
+                <mesh filename="package://neo_simulation/robots/mp_500/meshes/MP-500-WHEEL-RIGHT.dae" scale="0.001 0.001 0.001" />
+            </geometry>
+        </visual>
+        <collision>
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